File: BigBoard.brd (EAGLE design)
At the start: 28.9 x 39.4 mm, 12 parts

Commit message: I don't even
Parts:
- removed FRAME1: FRAME-LETTER, SparkFun-Aesthetics:CREATIVE_COMMONS
Changed lines of the file:
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@@
 <element name="J_OUTPUT" library="SparkFun-Connectors" package="MOLEX-1X6" value="" x="3.81" y="20.955" rot="R270"/>
 <element name="R1" library="SparkFun-Passives" package="0805" value="330" x="8.255" y="7.62" rot="R90"/>
-<element name="FRAME1" library="SparkFun-Aesthetics" package="CREATIVE_COMMONS" value="FRAME-LETTER" x="-77.47" y="24.13"/>
 <element name="J_DISPLAY" library="SparkFun-Connectors" package="2X5-SHROUDED" value="M05X2SHD" x="15.24" y="33.655" rot="R270"/>
 <element name="U$2" library="bigboard" package="A6278EA" value="A6278EA" x="15.24" y="15.875" rot="R90"/>

Commit message: Replace 0805 resistor with 0603
Parts:
- R1: value 330 -> (none); device SparkFun-Passives:0805 -> SparkFun-Passives:0603-RES
- moved R1 1.27 mm to (8.26, 6.35)
Routing:
- net N$13: track 3.59 -> 4.91 mm
Changed lines of the file:
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@@
 <element name="J_INPUT" library="SparkFun-Connectors" package="MOLEX-1X6" value="" x="25.4" y="8.255" rot="R90"/>
 <element name="J_OUTPUT" library="SparkFun-Connectors" package="MOLEX-1X6" value="" x="3.81" y="20.955" rot="R270"/>
-<element name="R1" library="SparkFun-Passives" package="0805" value="330" x="8.255" y="7.62" rot="R90"/>
 <element name="J_DISPLAY" library="SparkFun-Connectors" package="2X5-SHROUDED" value="M05X2SHD" x="15.24" y="33.655" rot="R270"/>
 <element name="U$2" library="bigboard" package="A6278EA" value="A6278EA" x="15.24" y="15.875" rot="R90"/>
@@
 <element name="STANDOFF3" library="SparkFun-Electromechanical" package="STAND-OFF" value="STAND-OFF" x="3.81" y="25.4"/>
 <element name="STANDOFF4" library="SparkFun-Electromechanical" package="STAND-OFF" value="STAND-OFF" x="25.4" y="25.4"/>
+<element name="R1" library="SparkFun-Passives" package="0603-RES" value="" x="8.255" y="6.35" rot="R90"/>
 </elements>
 <signals>
@@
 </signal>
 <signal name="GND">
-<contactref element="R1" pad="1"/>
 <contactref element="J_OUTPUT" pad="1"/>
 <contactref element="J_INPUT" pad="6"/>
@@
 <wire x1="19.05" y1="6.985" x2="19.05" y2="3.81" width="0.4064" layer="16"/>
 <wire x1="11.795" y1="2.54" x2="11.795" y2="3.18" width="0.4064" layer="1"/>
-<wire x1="11.795" y1="3.18" x2="8.255" y2="6.72" width="0.4064" layer="1"/>
 <wire x1="3.81" y1="20.955" x2="8.89" y2="15.875" width="0.4064" layer="1"/>
 <wire x1="8.89" y1="15.875" x2="13.97" y2="15.875" width="0.4064" layer="1"/>
 <wire x1="13.97" y1="15.875" x2="13.97" y2="4.715" width="0.4064" layer="1"/>
 <wire x1="13.97" y1="4.715" x2="11.795" y2="2.54" width="0.4064" layer="1"/>
+<contactref element="R1" pad="1"/>
+<wire x1="11.795" y1="2.54" x2="8.835" y2="5.5" width="0.4064" layer="1"/>
+<wire x1="8.835" y1="5.5" x2="8.255" y2="5.5" width="0.4064" layer="1"/>
 </signal>
 <signal name="SDO">
@@
 </signal>
 <signal name="N$13">
+<contactref element="U$2" pad="15"/>
+<wire x1="9.26" y1="9.525" x2="11.43" y2="9.525" width="0.4064" layer="1"/>
 <contactref element="R1" pad="2"/>
-<contactref element="U$2" pad="15"/>
-<wire x1="8.255" y1="8.52" x2="9.26" y2="9.525" width="0.4064" layer="1"/>
-<wire x1="9.26" y1="9.525" x2="11.43" y2="9.525" width="0.4064" layer="1"/>
+<wire x1="9.26" y1="9.525" x2="8.255" y2="8.52" width="0.4064" layer="1"/>
+<wire x1="8.255" y1="8.52" x2="8.255" y2="7.2" width="0.4064" layer="1"/>
 </signal>
 <signal name="VLED">
